Commit message: 修改livox_mid_360源码,令livox_mid_360支持ubuntu20.04+noetic

File: src/livox_laser_simulation/urdf/livox_mid360.xacro (robot description, xacro)
@@ -84,6 +84,6 @@
     <xacro:Livox_Mid_gazebo_sensor name="${name}" visualize="${visualize}"/>
   </xacro:macro>
-    <xacro:Livox_Mid40 name="livox"/>
+    <!-- <xacro:Livox_Mid40 name="livox"/>
   <xacro:include filename="$(find livox_laser_simulation)/urdf/standardrobots_oasis300.xacro"/>
-  <xacro:link_oasis name="oasis"/>
+  <xacro:link_oasis name="oasis"/> -->
 </robot>

File: src/my_robot_description/urdf/robot.xacro (robot description, xacro)
@@ -1,4 +1,5 @@
 <?xml version="1.0"?>
 <robot name="my_robot" xmlns:xacro="http://www.ros.org/wiki/xacro">
+  <!-- <xacro:include filename="$(find livox_laser_simulation)/urdf/livox_mid360.xacro"/> -->
   <!-- 参数定义 -->
   <xacro:property name="base_width" value="0.4"/>
@@ -116,4 +117,16 @@
     <origin xyz="0 0 0.5" rpy="0 0 0" />
   </VLP-16>
+  <!-- 1. 引入 Livox Mid-360 的宏定义文件 -->
+  <xacro:include filename="$(find livox_laser_simulation)/urdf/livox_mid360.xacro"/>
+  <!-- 2. 调用宏生成雷达 -->
+  <!-- 假设第一步查出来的宏名字叫 Livox_Mid_360，如果查出来叫别的，请把这里替换掉 -->
+  <xacro:Livox_Mid40 name="livox"/>
+  <!-- 3. 手动创建一个关节，把雷达绑在小车上 -->
+  <!-- 注意：Livox 生成的基座 link 名字通常是 "你的name参数_base"，也就是 "livox_base" -->
+  <joint name="livox_mount_joint" type="fixed">
+    <parent link="base_link"/>
+    <child link="livox_base"/>
+    <origin xyz="0.45 0.0 0.08" rpy="0 0 0" />
+  </joint>
   <!-- 3. Gazebo 差速驱动插件 -->
   <gazebo>

Commit message: 修改mid360代码适配个人小车

File: src/livox_laser_simulation/urdf/livox_mid360.xacro (robot description, xacro)
@@ -4,7 +4,7 @@
   <xacro:property name="laser_min_range" value="0.1"/>
   <xacro:property name="laser_max_range" value="200.0"/>
-  <xacro:property name="ros_topic" value="scan"/>
+  <xacro:property name="ros_topic" value="points_mid"/>
   <xacro:property name="samples" value="24000"/>
-  <xacro:property name="downsample" value="1"/>
+  <xacro:property name="downsample" value="2"/>
   <xacro:macro name="null_inertial">
     <inertial>
@@ -17,5 +17,5 @@
   <xacro:macro name="Livox_Mid_gazebo_sensor" params="visualize:=True update_rate:=10 resolution:=0.002 noise_mean:=0.0 noise_stddev:=0.01 name:=livox">
     <gazebo reference="${name}">
-      <sensor type="ray" name="laser_${name}">
+      <sensor type="ray" name="${name}">
         <pose>0 0 0 0 0 0</pose>
         <visualize>${visualize}</visualize>
@@ -74,16 +74,13 @@
       </collision>
     </link>
-    <link name="${name}">
+    <link name="laser_${name}">
       <xacro:null_inertial/>
     </link>
     <joint name="${name}_to_${name}_base_joint" type="fixed">
       <parent link="${name}_base"/>
-      <child link="${name}"/>
-      <origin rpy="0 0 0" xyz="0.0 1.0 0.2"/>
+      <child link="laser_${name}"/>
+      <origin rpy="0 0 0" xyz="0.0 0.0 0.2"/>
     </joint>
-    <xacro:Livox_Mid_gazebo_sensor name="${name}" visualize="${visualize}"/>
+    <xacro:Livox_Mid_gazebo_sensor name="laser_${name}" visualize="${visualize}"/>
   </xacro:macro>
-    <!-- <xacro:Livox_Mid40 name="livox"/>
-  <xacro:include filename="$(find livox_laser_simulation)/urdf/standardrobots_oasis300.xacro"/>
-  <xacro:link_oasis name="oasis"/> -->
 </robot>

File: src/my_robot_description/urdf/robot.xacro (robot description, xacro)
@@ -120,12 +120,11 @@
   <xacro:include filename="$(find livox_laser_simulation)/urdf/livox_mid360.xacro"/>
   <!-- 2. 调用宏生成雷达 -->
-  <!-- 假设第一步查出来的宏名字叫 Livox_Mid_360，如果查出来叫别的，请把这里替换掉 -->
   <xacro:Livox_Mid40 name="livox"/>
   <!-- 3. 手动创建一个关节，把雷达绑在小车上 -->
   <!-- 注意：Livox 生成的基座 link 名字通常是 "你的name参数_base"，也就是 "livox_base" -->
-  <joint name="livox_mount_joint" type="fixed">
+  <joint name="laser_livox_bridge_joint" type="fixed">
     <parent link="base_link"/>
     <child link="livox_base"/>
-    <origin xyz="0.45 0.0 0.08" rpy="0 0 0" />
+    <origin xyz="0.45 0.0 0.45" rpy="0 0 0" />
   </joint>
   <!-- 3. Gazebo 差速驱动插件 -->

Commit message: 彻底打通mid360+vlp16的融合

File: src/livox_laser_simulation/urdf/livox_mid360.xacro (robot description, xacro)
@@ -10,7 +10,7 @@
     <inertial>
       <mass value="0.1"/>
-    <inertia ixx="0.01" ixy="0" ixz="0"
-          iyy="0.01" iyz="0"
-          izz="0.01"/>
+      <inertia ixx="0.01" ixy="0" ixz="0"
+               iyy="0.01" iyz="0"
+               izz="0.01"/>
     </inertial>
   </xacro:macro>
@@ -21,65 +21,74 @@
         <visualize>${visualize}</visualize>
         <update_rate>${update_rate}</update_rate>
-        <!-- This ray plgin is only for visualization. -->
         <plugin name="gazebo_ros_laser_controller" filename="liblivox_laser_simulation.so">
-			<ray>
-			  <scan>
-				<horizontal>
-				<samples>100</samples>
-				<resolution>1</resolution>
-				<min_angle>${0}</min_angle>
-				<max_angle>${2*M_PI}</max_angle>
-				</horizontal>
-				<vertical>
-				<samples>360</samples>
-				<resolution>1</resolution>
-				<min_angle>${-7.22/180*M_PI}</min_angle>
-				<max_angle>${55.22/180*M_PI}</max_angle>
-				</vertical>
-			  </scan>
-			  <range>
-				<min>${laser_min_range}</min>
-				<max>${laser_max_range}</max>
-				<resolution>${resolution}</resolution>
-			  </range>
-			  <noise>
-				<type>gaussian</type>
-				<mean>${noise_mean}</mean>
-				<stddev>${noise_stddev}</stddev>
-			  </noise>
-			</ray>
+          <ray>
+            <scan>
+              <horizontal>
+                <samples>100</samples>
+                <resolution>1</resolution>
+                <min_angle>${0}</min_angle>
+                <max_angle>${2*M_PI}</max_angle>
+              </horizontal>
+              <vertical>
+                <samples>360</samples>
+                <resolution>1</resolution>
+                <min_angle>${-7.22/180*M_PI}</min_angle>
+                <max_angle>${55.22/180*M_PI}</max_angle>
+              </vertical>
+            </scan>
+            <range>
+              <min>${laser_min_range}</min>
+              <max>${laser_max_range}</max>
+              <resolution>${resolution}</resolution>
+            </range>
+            <noise>
+              <type>gaussian</type>
+              <mean>${noise_mean}</mean>
+              <stddev>${noise_stddev}</stddev>
+            </noise>
+          </ray>
           <visualize>${visualize}</visualize>
-		  <samples>${samples}</samples>
-		  <downsample>${downsample}</downsample>
-		  <csv_file_name>package://livox_laser_simulation/scan_mode/mid360.csv</csv_file_name>
-		  <ros_topic>${ros_topic}</ros_topic>
+          <samples>${samples}</samples>
+          <downsample>${downsample}</downsample>
+          <csv_file_name>package://livox_laser_simulation/scan_mode/mid360.csv</csv_file_name>
+          <ros_topic>${ros_topic}</ros_topic>
         </plugin>
       </sensor>
     </gazebo>
   </xacro:macro>
-  <xacro:macro name="Livox_Mid40" params="visualize:=True name:=livox">
-    <link name="${name}_base">
+  <!--
+    Livox Mid-360 URDF 宏
+    参数:
+      name      - 雷达名称前缀 (默认 livox)
+      parent    - 父 link (默认 base_link)
+      xyz       - 安装位置偏移 (默认 "0.45 0 0.45")
+      rpy       - 安装姿态 (默认 "0 0 0")
+      visualize - 是否在 Gazebo 中可视化 (默认 true)
+    结构: parent → laser_${name} (直接挂载，无中间 link)
+  -->
+  <xacro:macro name="Livox_Mid40" params="visualize:=True name:=livox parent:=base_link xyz:='0.45 0 0.45' rpy:='0 0 0'">
+    <!-- 传感器 link (带 mesh visual) -->
+    <link name="laser_${name}">
       <xacro:null_inertial/>
       <visual>
-        <origin xyz="0.00 0 0.0" rpy="0 0 0"/>
+        <origin xyz="0 0 0" rpy="0 0 0"/>
         <geometry>
-          <mesh filename="package://livox_laser_simulation/meshes/livox_mid40.dae">
-          </mesh>
+          <mesh filename="package://livox_laser_simulation/meshes/livox_mid40.dae"/>
         </geometry>
       </visual>
       <collision>
-		  <origin xyz="0 0 0" rpy="0 0 0" /> <geometry> <mesh
-		  filename="package://livox_laser_simulation/meshes/livox_mid40.dae">
-		  </mesh> </geometry>
+        <origin xyz="0 0 0" rpy="0 0 0"/>
+        <geometry>
+          <mesh filename="package://livox_laser_simulation/meshes/livox_mid40.dae"/>
+        </geometry>
       </collision>
     </link>
-    <link name="laser_${name}">
-      <xacro:null_inertial/>
-    </link>
-    <joint name="${name}_to_${name}_base_joint" type="fixed">
-      <parent link="${name}_base"/>
+    <!-- 固定关节: 父 link → 传感器 (直接挂载) -->
+    <joint name="${name}_mount_joint" type="fixed">
+      <parent link="${parent}"/>
       <child link="laser_${name}"/>
-      <origin rpy="0 0 0" xyz="0.0 0.0 0.2"/>
+      <origin xyz="${xyz}" rpy="${rpy}"/>
     </joint>
+    <!-- Gazebo 传感器插件 -->
     <xacro:Livox_Mid_gazebo_sensor name="laser_${name}" visualize="${visualize}"/>
   </xacro:macro>

File: src/my_robot_description/urdf/robot.xacro (robot description, xacro)
@@ -119,12 +119,6 @@
   <!-- 1. 引入 Livox Mid-360 的宏定义文件 -->
   <xacro:include filename="$(find livox_laser_simulation)/urdf/livox_mid360.xacro"/>
-  <!-- 2. 调用宏生成雷达 -->
-  <xacro:Livox_Mid40 name="livox"/>
-  <!-- 3. 手动创建一个关节，把雷达绑在小车上 -->
-  <joint name="laser_livox_bridge_joint" type="fixed">
-    <parent link="base_link"/>
-    <child link="livox_base"/>
-    <origin xyz="0.45 0.0 0.45" rpy="0 0 0" />
-  </joint>
+  <!-- 2. 调用宏生成雷达 (直接指定 parent 和安装位置) -->
+  <xacro:Livox_Mid40 name="livox" parent="base_link" xyz="0.45 0 0.45" rpy="3.1415926 0 0"/>
   <!-- 3. Gazebo 差速驱动插件 -->
   <gazebo>
@@ -144,5 +138,5 @@
       <robotBaseFrame>base_link</robotBaseFrame>
       <!-- 补充这些参数 -->
-      <publishWheelTF>true</publishWheelTF>
+      <publishWheelTF>false</publishWheelTF>
       <publishOdomTF>true</publishOdomTF>
       <publishWheelJointState>true</publishWheelJointState>
