Commit message: 修改模型

File: src/my_robot_description/urdf/robot.xacro (robot description, xacro)
@@ -42,5 +42,5 @@
       <parent link="base_link"/>
       <child link="${prefix}_wheel"/>
-      <origin xyz="0 ${reflect * (base_width/2 + wheel_width/2)} -0.05" rpy="-1.57 0 0"/>
+      <origin xyz="-0.05 ${reflect * (base_width/2 + wheel_width/2)} -0.05" rpy="-1.57 0 0"/>
       <axis xyz="0 0 1"/>
     </joint>

Commit message: 修改模型

File: src/my_robot_description/urdf/robot.xacro (robot description, xacro)
@@ -3,5 +3,5 @@
   <!-- 参数定义 -->
   <xacro:property name="base_width" value="0.4"/>
-  <xacro:property name="base_length" value="0.5"/>
+  <xacro:property name="base_length" value="1.0"/>
   <xacro:property name="wheel_radius" value="0.1"/>
   <xacro:property name="wheel_width" value="0.05"/>
@@ -42,5 +42,5 @@
       <parent link="base_link"/>
       <child link="${prefix}_wheel"/>
-      <origin xyz="-0.05 ${reflect * (base_width/2 + wheel_width/2)} -0.05" rpy="-1.57 0 0"/>
+      <origin xyz="-0.2 ${reflect * (base_width/2 + wheel_width/2)} -0.05" rpy="-1.57 0 0"/>
       <axis xyz="0 0 1"/>
     </joint>
@@ -64,5 +64,5 @@
     <parent link="base_link"/>
     <child link="caster_wheel"/>
-    <origin xyz="0.2 0 -0.1" rpy="0 0 0"/>
+    <origin xyz="0.4 0 -0.1" rpy="0 0 0"/>
   </joint>
   <!-- 给万向轮设置摩擦力 (Gazebo 专用) -->
@@ -75,4 +75,5 @@
     <plugin name="differential_drive_controller" filename="libgazebo_ros_diff_drive.so">
       <legacyMode>false</legacyMode>
+      <rosDebugLevel>na</rosDebugLevel>
       <alwaysOn>true</alwaysOn>
       <updateRate>20</updateRate>
@@ -86,4 +87,12 @@
       <odometryFrame>odom</odometryFrame>
       <robotBaseFrame>base_link</robotBaseFrame>
+      <!-- 补充这些参数 -->
+      <publishWheelTF>true</publishWheelTF>
+      <publishOdomTF>true</publishOdomTF>
+      <publishWheelJointState>true</publishWheelJointState>
+      <wheelAcceleration>1.0</wheelAcceleration>
+      <wheelTorque>20</wheelTorque>
+      <odometrySource>world</odometrySource>
+      <publishTf>1</publishTf>
     </plugin>
   </gazebo>

Commit message: 修改模型,增加激光雷达到车体上

File: src/my_robot_description/urdf/robot.xacro (robot description, xacro)
@@ -71,4 +71,22 @@
     <mu2>0.0</mu2>
   </gazebo>
+    <!-- 激光雷达 Link -->
+  <link name="laser_link">
+    <visual>
+      <geometry> <cylinder radius="0.03" length="0.05"/> </geometry>
+      <material name="black"/>
+    </visual>
+    <collision>
+      <geometry> <cylinder radius="0.03" length="0.05"/> </geometry>
+    </collision>
+    <xacro:default_inertial mass="0.1"/>
+  </link>
+  <!-- 激光雷达 Joint -->
+  <joint name="laser_joint" type="fixed">
+    <parent link="base_link"/>
+    <child link="laser_link"/>
+    <!-- 放在底盘上方 (base_z + 0.05/2) -->
+    <origin xyz="0 0 0.075" rpy="0 0 0"/>
+  </joint>
   <!-- 3. Gazebo 差速驱动插件 -->
   <gazebo>
@@ -97,3 +115,29 @@
     </plugin>
   </gazebo>
+    <gazebo reference="laser_link">
+        <sensor type="ray" name="head_hokuyo_sensor">
+        <pose>0 0 0 0 0 0</pose>
+        <visualize>true</visualize> <!-- 设置为 true，你就能在 Gazebo 里看到扫描线 -->
+        <update_rate>40</update_rate>
+        <ray>
+            <scan>
+            <horizontal>
+                <samples>720</samples>
+                <resolution>1</resolution>
+                <min_angle>-1.570796</min_angle>
+                <max_angle>1.570796</max_angle>
+            </horizontal>
+            </scan>
+            <range>
+            <min>0.10</min>
+            <max>30.0</max>
+            <resolution>0.01</resolution>
+            </range>
+        </ray>
+        <plugin name="gazebo_ros_head_hokuyo_controller" filename="libgazebo_ros_laser.so">
+            <topicName>/scan</topicName>
+            <frameName>laser_link</frameName>
+        </plugin>
+        </sensor>
+    </gazebo>
 </robot>

Commit message: 消除控制警告,解决base_link的惯性量问题

File: src/my_robot_description/urdf/robot.xacro (robot description, xacro)
@@ -16,4 +16,10 @@
     </inertial>
   </xacro:macro>
+  <link name="base_footprint"/>
+  <joint name="base_joint" type="fixed">
+    <parent link="base_footprint"/>
+    <child link="base_link"/>
+    <origin xyz="0 0 0.1" rpy="0 0 0"/>
+  </joint>
   <!-- 1. 底盘 -->
   <link name="base_link">

Commit message: 添加velodyne雷达包,增加16线雷达到模型上

File: src/my_robot_description/urdf/robot.xacro (robot description, xacro)
@@ -95,4 +95,25 @@
     <origin xyz="0 0 0.075" rpy="0 0 0"/>
   </joint>
+  <link name="velodyne_base_link">
+    <inertial>
+      <mass value="0.83"/>
+      <inertia ixx="0.000908" ixy="0" ixz="0" iyy="0.000908" iyz="0" izz="0.001104"/>
+    </inertial>
+    <visual>
+      <geometry>
+        <cylinder length="0.0717" radius="0.0516"/>
+      </geometry>
+      <material name="black"/>
+    </visual>
+  </link>
+  <joint name="velodyne_base_mount_joint" type="fixed">
+    <parent link="base_link"/>
+    <child link="velodyne_base_link"/>
+    <origin xyz="0 0 0.5" rpy="0 0 0"/>
+  </joint>
+  <!-- 显式传入参数 -->
+  <VLP-16 parent="base_link" name="velodyne" topic="/velodyne_points" hz="10" samples="440" gpu="true">
+    <origin xyz="0 0 0.5" rpy="0 0 0" />
+  </VLP-16>
   <!-- 3. Gazebo 差速驱动插件 -->
   <gazebo>
@@ -124,5 +145,5 @@
     <sensor type="ray" name="head_hokuyo_sensor">
       <pose>0 0 0 0 0 0</pose>
-      <visualize>true</visualize>
+      <visualize>false</visualize>
       <update_rate>40</update_rate> <!-- 更新频率，越高越平滑，但越占CPU -->
       <ray>
@@ -154,3 +175,38 @@
     </sensor>
   </gazebo>
+  <!-- 确保 Gazebo 传感器配置正确挂载到 velodyne_base_link -->
+  <gazebo reference="velodyne_base_link">
+    <sensor type="ray" name="velodyne-VLP16">
+      <pose>0 0 0 0 0 0</pose>
+      <visualize>false</visualize>
+      <update_rate>10</update_rate>
+      <ray>
+        <scan>
+          <horizontal>
+            <samples>440</samples>
+            <resolution>1</resolution>
+            <min_angle>-3.14159</min_angle>
+            <max_angle>3.14159</max_angle>
+          </horizontal>
+          <vertical>
+            <samples>16</samples>
+            <min_angle>-0.261799</min_angle>
+            <max_angle>0.261799</max_angle>
+          </vertical>
+        </scan>
+        <range>
+          <min>0.3</min>
+          <max>130.0</max>
+          <resolution>0.001</resolution>
+        </range>
+      </ray>
+      <plugin name="gazebo_ros_velodyne_laser_controller" filename="libgazebo_ros_velodyne_laser.so">
+        <topicName>/velodyne_points</topicName>
+        <frameName>velodyne_base_link</frameName>
+        <min_range>0.9</min_range>
+        <max_range>130.0</max_range>
+        <gaussianNoise>0.008</gaussianNoise>
+      </plugin>
+    </sensor>
+  </gazebo>
 </robot>

Commit message: 修改16线高度

File: src/my_robot_description/urdf/robot.xacro (robot description, xacro)
@@ -115,5 +115,5 @@
   <!-- 显式传入参数 -->
   <VLP-16 parent="base_link" name="velodyne" topic="/velodyne_points" hz="10" samples="440" gpu="true">
-    <origin xyz="0 0 0.5" rpy="0 0 0" />
+    <origin xyz="0 0 0.3" rpy="0 0 0" />
   </VLP-16>
   <!-- 1. 引入 Livox Mid-360 的宏定义文件 -->

Commit message: 增加单线雷达,修改车辆传感器位置

File: src/my_robot_description/urdf/robot.xacro (robot description, xacro)
@@ -1,5 +1,4 @@
 <?xml version="1.0"?>
 <robot name="my_robot" xmlns:xacro="http://www.ros.org/wiki/xacro">
-  <!-- <xacro:include filename="$(find livox_laser_simulation)/urdf/livox_mid360.xacro"/> -->
   <!-- 参数定义 -->
   <xacro:property name="base_width" value="0.4"/>
@@ -10,5 +9,5 @@
   <material name="blue"> <color rgba="0 0 0.8 1"/> </material>
   <material name="black"> <color rgba="0 0 0 1"/> </material>
-  <!-- 惯性矩阵宏 (Gazebo仿真必备，否则模型会乱飞) -->
+  <!-- 惯性矩阵宏 -->
   <xacro:macro name="default_inertial" params="mass">
     <inertial>
@@ -56,5 +55,5 @@
   <xacro:wheel prefix="left" reflect="1"/>
   <xacro:wheel prefix="right" reflect="-1"/>
-    <!-- 添加支撑脚 (万向轮) -->
+  <!-- 3. 添加支撑脚 (万向轮) -->
   <link name="caster_wheel">
     <visual>
@@ -67,5 +66,4 @@
     <xacro:default_inertial mass="0.5"/>
   </link>
-  <!-- 支撑脚关节 (固定连接) -->
   <joint name="caster_joint" type="fixed">
     <parent link="base_link"/>
@@ -73,27 +71,72 @@
     <origin xyz="0.4 0 -0.1" rpy="0 0 0"/>
   </joint>
-  <!-- 给万向轮设置摩擦力 (Gazebo 专用) -->
   <gazebo reference="caster_wheel">
     <mu1>0.0</mu1>
     <mu2>0.0</mu2>
   </gazebo>
-    <!-- 激光雷达 Link -->
-  <link name="laser_link">
-    <visual>
-      <geometry> <cylinder radius="0.03" length="0.05"/> </geometry>
-      <material name="black"/>
-    </visual>
-    <collision>
-      <geometry> <cylinder radius="0.03" length="0.05"/> </geometry>
-    </collision>
-    <xacro:default_inertial mass="0.1"/>
-  </link>
-  <!-- 激光雷达 Joint -->
-  <joint name="laser_joint" type="fixed">
-    <parent link="base_link"/>
-    <child link="laser_link"/>
-    <!-- 放在底盘上方 (base_z + 0.05/2) -->
-    <origin xyz="0 0 0.075" rpy="0 0 0"/>
-  </joint>
+  <!-- ========================================================== -->
+  <!-- 4. 四个单线激光雷达 (利用宏定义减少重复代码) -->
+  <!-- ========================================================== -->
+  <xacro:macro name="corner_laser" params="prefix x y z yaw">
+    <link name="${prefix}_laser_link">
+      <visual>
+        <geometry> <cylinder radius="0.03" length="0.05"/> </geometry>
+        <material name="black"/>
+      </visual>
+      <collision>
+        <geometry> <cylinder radius="0.03" length="0.05"/> </geometry>
+      </collision>
+      <xacro:default_inertial mass="0.1"/>
+    </link>
+    <joint name="${prefix}_laser_joint" type="fixed">
+      <parent link="base_link"/>
+      <child link="${prefix}_laser_link"/>
+      <!-- yaw 角度偏转使得雷达盲区朝向车体内部，视野最大化 -->
+      <origin xyz="${x} ${y} ${z}" rpy="0 0 ${yaw}"/>
+    </joint>
+    <gazebo reference="${prefix}_laser_link">
+      <sensor type="ray" name="${prefix}_hokuyo_sensor">
+        <pose>0 0 0 0 0 0</pose>
+        <visualize>false</visualize>
+        <update_rate>40</update_rate>
+        <ray>
+          <scan>
+            <horizontal>
+              <samples>720</samples>
+              <resolution>1</resolution>
+              <min_angle>-3.1415926</min_angle>
+              <max_angle>3.1415926</max_angle>
+            </horizontal>
+          </scan>
+          <range>
+            <min>0.10</min>
+            <max>10.0</max>
+            <resolution>0.01</resolution>
+          </range>
+          <noise>
+            <type>gaussian</type>
+            <mean>0.0</mean>
+            <stddev>0.01</stddev>
+          </noise>
+        </ray>
+        <plugin name="gazebo_ros_${prefix}_laser" filename="libgazebo_ros_laser.so">
+          <!-- 自动生成独立话题名，例如 /scan_fl, /scan_fr -->
+          <topicName>/scan_${prefix}</topicName>
+          <frameName>${prefix}_laser_link</frameName>
+          <rosDebugLevel>na</rosDebugLevel>
+        </plugin>
+      </sensor>
+    </gazebo>
+  </xacro:macro>
+  <!-- 部署四个单线雷达 (前左、前右、后左、后右) -->
+  <!-- 坐标计算: 长1.0的一半是0.5, 宽0.4的一半是0.2, 放在底盘上方z=0.075 -->
+  <!-- yaw 角度: 45度角(0.785rad)等，保证扫描盲区在车内部 -->
+  <xacro:corner_laser prefix="left" x="0.5" y="0.2" z="0.075" yaw="0.785" />
+  <xacro:corner_laser prefix="right" x="0.5" y="-0.2" z="0.075" yaw="-0.785" />
+  <xacro:corner_laser prefix="bleft" x="-0.5" y="0.2" z="0.075" yaw="2.356" />
+  <xacro:corner_laser prefix="bright" x="-0.5" y="-0.2" z="0.075" yaw="-2.356" />
+  <!-- ========================================================== -->
+  <!-- 5. 16线激光雷达 (车辆中心偏前0.3m) -->
+  <!-- ========================================================== -->
   <link name="velodyne_base_link">
     <inertial>
@@ -108,77 +151,14 @@
     </visual>
   </link>
+  <!-- 原代码z为0.5/0.3有点混乱，现统一放置在 x=0.3, y=0, z=0.3 处 -->
   <joint name="velodyne_base_mount_joint" type="fixed">
     <parent link="base_link"/>
     <child link="velodyne_base_link"/>
-    <origin xyz="0 0 0.5" rpy="0 0 0"/>
+    <origin xyz="0.3 0 0.8" rpy="0 0 0"/>
   </joint>
   <!-- 显式传入参数 -->
-  <VLP-16 parent="base_link" name="velodyne" topic="/velodyne_points" hz="10" samples="440" gpu="true">
-    <origin xyz="0 0 0.3" rpy="0 0 0" />
+  <VLP-16 parent="base_link" name="velodyne" topic="/points_16" hz="10" samples="440" gpu="true">
+    <origin xyz="0.3 0 0.3" rpy="0 0 0" />
   </VLP-16>
-  <!-- 1. 引入 Livox Mid-360 的宏定义文件 -->
-  <xacro:include filename="$(find livox_laser_simulation)/urdf/livox_mid360.xacro"/>
-  <!-- 2. 调用宏生成雷达 (直接指定 parent 和安装位置) -->
-  <xacro:Livox_Mid40 name="livox" parent="base_link" xyz="0.45 0 0.45" rpy="3.1415926 0 0"/>
-  <!-- 3. Gazebo 差速驱动插件 -->
-  <gazebo>
-    <plugin name="differential_drive_controller" filename="libgazebo_ros_diff_drive.so">
-      <legacyMode>false</legacyMode>
-      <rosDebugLevel>na</rosDebugLevel>
-      <alwaysOn>true</alwaysOn>
-      <updateRate>20</updateRate>
-      <leftJoint>left_wheel_joint</leftJoint>
-      <rightJoint>right_wheel_joint</rightJoint>
-      <wheelSeparation>${base_width + wheel_width}</wheelSeparation>
-      <wheelDiameter>${2 * wheel_radius}</wheelDiameter>
-      <torque>20</torque>
-      <commandTopic>cmd_vel</commandTopic>
-      <odometryTopic>odom</odometryTopic>
-      <odometryFrame>odom</odometryFrame>
-      <robotBaseFrame>base_link</robotBaseFrame>
-      <!-- 补充这些参数 -->
-      <publishWheelTF>false</publishWheelTF>
-      <publishOdomTF>true</publishOdomTF>
-      <publishWheelJointState>true</publishWheelJointState>
-      <wheelAcceleration>1.0</wheelAcceleration>
-      <wheelTorque>20</wheelTorque>
-      <odometrySource>world</odometrySource>
-      <publishTf>1</publishTf>
-    </plugin>
-  </gazebo>
-  <gazebo reference="laser_link">
-    <sensor type="ray" name="head_hokuyo_sensor">
-      <pose>0 0 0 0 0 0</pose>
-      <visualize>false</visualize>
-      <update_rate>40</update_rate> <!-- 更新频率，越高越平滑，但越占CPU -->
-      <ray>
-        <scan>
-          <horizontal>
-            <samples>720</samples>      <!-- 扫描点数，720通常对应0.5度分辨率 -->
-            <resolution>1</resolution>
-            <min_angle>-3.1415926</min_angle>
-            <max_angle>3.1415926</max_angle>
-          </horizontal>
-        </scan>
-        <range>
-          <min>0.10</min>               <!-- 盲区：小于此距离视为无效 -->
-          <max>10.0</max>               <!-- 测量上限 -->
-          <resolution>0.01</resolution> <!-- 测距精度 -->
-        </range>
-        <!-- 添加噪声模型，仿真环境下的必备，否则SLAM效果太理想 -->
-        <noise>
-          <type>gaussian</type>
-          <mean>0.0</mean>
-          <stddev>0.01</stddev>         <!-- 标准差，模拟0.01米的测量波动 -->
-        </noise>
-      </ray>
-      <plugin name="gazebo_ros_head_hokuyo_controller" filename="libgazebo_ros_laser.so">
-        <topicName>/scan</topicName>
-        <frameName>laser_link</frameName>
-        <rosDebugLevel>na</rosDebugLevel>
-      </plugin>
-    </sensor>
-  </gazebo>
-  <!-- 确保 Gazebo 传感器配置正确挂载到 velodyne_base_link -->
   <gazebo reference="velodyne_base_link">
     <sensor type="ray" name="velodyne-VLP16">
@@ -215,3 +195,36 @@
     </sensor>
   </gazebo>
+  <!-- ========================================================== -->
+  <!-- 6. Livox Mid-360 雷达 (车头中心点偏后0.1m) -->
+  <!-- ========================================================== -->
+  <xacro:include filename="$(find livox_laser_simulation)/urdf/livox_mid360.xacro"/>
+  <!-- 车头为 x=0.5, 往后偏0.1m，所以 x=0.4 -->
+  <xacro:Livox_Mid40 name="livox" parent="base_link" xyz="0.4 0 0.45" rpy="3.1415926 0 0"/>
+  <!-- ========================================================== -->
+  <!-- 7. 差速驱动底盘插件 -->
+  <!-- ========================================================== -->
+  <gazebo>
+    <plugin name="differential_drive_controller" filename="libgazebo_ros_diff_drive.so">
+      <legacyMode>false</legacyMode>
+      <rosDebugLevel>na</rosDebugLevel>
+      <alwaysOn>true</alwaysOn>
+      <updateRate>20</updateRate>
+      <leftJoint>left_wheel_joint</leftJoint>
+      <rightJoint>right_wheel_joint</rightJoint>
+      <wheelSeparation>${base_width + wheel_width}</wheelSeparation>
+      <wheelDiameter>${2 * wheel_radius}</wheelDiameter>
+      <torque>20</torque>
+      <commandTopic>cmd_vel</commandTopic>
+      <odometryTopic>odom</odometryTopic>
+      <odometryFrame>odom</odometryFrame>
+      <robotBaseFrame>base_link</robotBaseFrame>
+      <publishWheelTF>false</publishWheelTF>
+      <publishOdomTF>true</publishOdomTF>
+      <publishWheelJointState>true</publishWheelJointState>
+      <wheelAcceleration>1.0</wheelAcceleration>
+      <wheelTorque>20</wheelTorque>
+      <odometrySource>world</odometrySource>
+      <publishTf>1</publishTf>
+    </plugin>
+  </gazebo>
 </robot>
