Commit message: 修改16线雷达,避免16线雷达写法错误导致的gazebo崩溃

File: src/my_robot_description/urdf/robot.xacro (robot description, xacro)
@@ -1,68 +1,94 @@
 <?xml version="1.0"?>
 <robot name="my_robot" xmlns:xacro="http://www.ros.org/wiki/xacro">
-  <!-- 参数定义 -->
+  <!-- ============ 参数定义 ============ -->
   <xacro:property name="base_width" value="0.4"/>
   <xacro:property name="base_length" value="1.0"/>
+  <xacro:property name="base_height" value="0.1"/>
   <xacro:property name="wheel_radius" value="0.1"/>
   <xacro:property name="wheel_width" value="0.05"/>
-  <!-- 颜色宏 -->
-  <material name="blue"> <color rgba="0 0 0.8 1"/> </material>
-  <material name="black"> <color rgba="0 0 0 1"/> </material>
-  <!-- 惯性矩阵宏 -->
-  <xacro:macro name="default_inertial" params="mass">
+  <!-- ============ 惯性矩阵宏 ============ -->
+  <xacro:macro name="box_inertial" params="mass x y z">
     <inertial>
+      <origin xyz="0 0 0" rpy="0 0 0"/>
       <mass value="${mass}"/>
-      <inertia ixx="0.01" ixy="0.0" ixz="0.0" iyy="0.01" iyz="0.0" izz="0.01"/>
+      <inertia ixx="${mass*(y*y+z*z)/12}" ixy="0" ixz="0"
+               iyy="${mass*(x*x+z*z)/12}" iyz="0"
+               izz="${mass*(x*x+y*y)/12}"/>
     </inertial>
   </xacro:macro>
+  <xacro:macro name="cylinder_inertial" params="mass radius length">
+    <inertial>
+      <origin xyz="0 0 0" rpy="0 0 0"/>
+      <mass value="${mass}"/>
+      <inertia ixx="${mass*(3*radius*radius+length*length)/12}" ixy="0" ixz="0"
+               iyy="${mass*(3*radius*radius+length*length)/12}" iyz="0"
+               izz="${mass*radius*radius/2}"/>
+    </inertial>
+  </xacro:macro>
+  <xacro:macro name="sphere_inertial" params="mass radius">
+    <inertial>
+      <origin xyz="0 0 0" rpy="0 0 0"/>
+      <mass value="${mass}"/>
+      <inertia ixx="${2*mass*radius*radius/5}" ixy="0" ixz="0"
+               iyy="${2*mass*radius*radius/5}" iyz="0"
+               izz="${2*mass*radius*radius/5}"/>
+    </inertial>
+  </xacro:macro>
+  <!-- ============ base_footprint ============ -->
   <link name="base_footprint"/>
   <joint name="base_joint" type="fixed">
     <parent link="base_footprint"/>
     <child link="base_link"/>
-    <origin xyz="0 0 0.1" rpy="0 0 0"/>
+    <origin xyz="0 0 0.15" rpy="0 0 0"/>
   </joint>
-  <!-- 1. 底盘 -->
+  <!-- ============ 1. 底盘 ============ -->
   <link name="base_link">
     <visual>
-      <geometry> <box size="${base_length} ${base_width} 0.1"/> </geometry>
-      <material name="blue"/>
+      <origin xyz="0 0 0" rpy="0 0 0"/>
+      <geometry><box size="${base_length} ${base_width} ${base_height}"/></geometry>
+      <material name="blue"><color rgba="0 0 0.8 1"/></material>
     </visual>
     <collision>
-      <geometry> <box size="${base_length} ${base_width} 0.1"/> </geometry>
+      <origin xyz="0 0 0" rpy="0 0 0"/>
+      <geometry><box size="${base_length} ${base_width} ${base_height}"/></geometry>
     </collision>
-    <xacro:default_inertial mass="5.0"/>
+    <xacro:box_inertial mass="5.0" x="${base_length}" y="${base_width}" z="${base_height}"/>
   </link>
-  <!-- 2. 轮子宏 -->
+  <!-- ============ 2. 轮子宏 ============ -->
   <xacro:macro name="wheel" params="prefix reflect">
     <link name="${prefix}_wheel">
       <visual>
-        <geometry> <cylinder radius="${wheel_radius}" length="${wheel_width}"/> </geometry>
-        <material name="black"/>
+        <origin xyz="0 0 0" rpy="0 0 0"/>
+        <geometry><cylinder radius="${wheel_radius}" length="${wheel_width}"/></geometry>
+        <material name="black"><color rgba="0 0 0 1"/></material>
       </visual>
       <collision>
-        <geometry> <cylinder radius="${wheel_radius}" length="${wheel_width}"/> </geometry>
+        <origin xyz="0 0 0" rpy="0 0 0"/>
+        <geometry><cylinder radius="${wheel_radius}" length="${wheel_width}"/></geometry>
       </collision>
-      <xacro:default_inertial mass="1.0"/>
+      <xacro:cylinder_inertial mass="1.0" radius="${wheel_radius}" length="${wheel_width}"/>
     </link>
     <joint name="${prefix}_wheel_joint" type="continuous">
       <parent link="base_link"/>
       <child link="${prefix}_wheel"/>
-      <origin xyz="-0.2 ${reflect * (base_width/2 + wheel_width/2)} -0.05" rpy="-1.57 0 0"/>
+      <origin xyz="-0.2 ${reflect * (base_width/2 + wheel_width/2)} -0.05" rpy="-1.5708 0 0"/>
       <axis xyz="0 0 1"/>
+      <limit lower="-100" upper="100" effort="20" velocity="10"/>
     </joint>
   </xacro:macro>
-  <!-- 调用轮子宏 -->
   <xacro:wheel prefix="left" reflect="1"/>
   <xacro:wheel prefix="right" reflect="-1"/>
-  <!-- 3. 添加支撑脚 (万向轮) -->
+  <!-- ============ 3. 万向轮 ============ -->
   <link name="caster_wheel">
     <visual>
-      <geometry> <sphere radius="0.05"/> </geometry>
+      <origin xyz="0 0 0" rpy="0 0 0"/>
+      <geometry><sphere radius="0.05"/></geometry>
       <material name="black"/>
     </visual>
     <collision>
-      <geometry> <sphere radius="0.05"/> </geometry>
+      <origin xyz="0 0 0" rpy="0 0 0"/>
+      <geometry><sphere radius="0.05"/></geometry>
     </collision>
-    <xacro:default_inertial mass="0.5"/>
+    <xacro:sphere_inertial mass="0.5" radius="0.05"/>
   </link>
   <joint name="caster_joint" type="fixed">
@@ -75,22 +101,21 @@
     <mu2>0.0</mu2>
   </gazebo>
-  <!-- ========================================================== -->
-  <!-- 4. 四个单线激光雷达 (利用宏定义减少重复代码) -->
-  <!-- ========================================================== -->
+  <!-- ============ 4. 四个单线激光雷达 ============ -->
   <xacro:macro name="corner_laser" params="prefix x y z yaw">
     <link name="${prefix}_laser_link">
       <visual>
-        <geometry> <cylinder radius="0.03" length="0.05"/> </geometry>
+        <origin xyz="0 0 0" rpy="0 0 0"/>
+        <geometry><cylinder radius="0.03" length="0.05"/></geometry>
         <material name="black"/>
       </visual>
       <collision>
-        <geometry> <cylinder radius="0.03" length="0.05"/> </geometry>
+        <origin xyz="0 0 0" rpy="0 0 0"/>
+        <geometry><cylinder radius="0.03" length="0.05"/></geometry>
       </collision>
-      <xacro:default_inertial mass="0.1"/>
+      <xacro:cylinder_inertial mass="0.1" radius="0.03" length="0.05"/>
     </link>
     <joint name="${prefix}_laser_joint" type="fixed">
       <parent link="base_link"/>
       <child link="${prefix}_laser_link"/>
-      <!-- yaw 角度偏转使得雷达盲区朝向车体内部，视野最大化 -->
       <origin xyz="${x} ${y} ${z}" rpy="0 0 ${yaw}"/>
     </joint>
@@ -121,5 +146,4 @@
         </ray>
         <plugin name="gazebo_ros_${prefix}_laser" filename="libgazebo_ros_laser.so">
-          <!-- 自动生成独立话题名，例如 /scan_fl, /scan_fr -->
           <topicName>/scan_${prefix}</topicName>
           <frameName>${prefix}_laser_link</frameName>
@@ -129,38 +153,24 @@
     </gazebo>
   </xacro:macro>
-  <!-- 部署四个单线雷达 (前左、前右、后左、后右) -->
-  <!-- 坐标计算: 长1.0的一半是0.5, 宽0.4的一半是0.2, 放在底盘上方z=0.075 -->
-  <!-- yaw 角度: 45度角(0.785rad)等，保证扫描盲区在车内部 -->
-  <xacro:corner_laser prefix="left" x="0.5" y="0.2" z="0.075" yaw="0.785" />
-  <xacro:corner_laser prefix="right" x="0.5" y="-0.2" z="0.075" yaw="-0.785" />
-  <xacro:corner_laser prefix="bleft" x="-0.5" y="0.2" z="0.075" yaw="2.356" />
-  <xacro:corner_laser prefix="bright" x="-0.5" y="-0.2" z="0.075" yaw="-2.356" />
-  <!-- ========================================================== -->
-  <!-- 5. 16线激光雷达 (车辆中心偏前0.3m) -->
-  <!-- ========================================================== -->
+  <xacro:corner_laser prefix="left"    x="0.5"  y="0.2"  z="0.075" yaw="0.785" />
+  <xacro:corner_laser prefix="right"   x="0.5"  y="-0.2" z="0.075" yaw="-0.785" />
+  <xacro:corner_laser prefix="bleft"   x="-0.5" y="0.2"  z="0.075" yaw="2.356" />
+  <xacro:corner_laser prefix="bright"  x="-0.5" y="-0.2" z="0.075" yaw="-2.356" />
+  <!-- ============ 5. 16线激光雷达 (使用 GPU 版本 Velodyne 插件) ============ -->
   <link name="velodyne_base_link">
-    <inertial>
-      <mass value="0.83"/>
-      <inertia ixx="0.000908" ixy="0" ixz="0" iyy="0.000908" iyz="0" izz="0.001104"/>
-    </inertial>
+    <xacro:cylinder_inertial mass="0.83" radius="0.0516" length="0.0717"/>
     <visual>
-      <geometry>
-        <cylinder length="0.0717" radius="0.0516"/>
-      </geometry>
+      <origin xyz="0 0 0" rpy="0 0 0"/>
+      <geometry><cylinder length="0.0717" radius="0.0516"/></geometry>
       <material name="black"/>
     </visual>
   </link>
-  <!-- 原代码z为0.5/0.3有点混乱，现统一放置在 x=0.3, y=0, z=0.3 处 -->
   <joint name="velodyne_base_mount_joint" type="fixed">
     <parent link="base_link"/>
     <child link="velodyne_base_link"/>
-    <origin xyz="0.3 0 0.8" rpy="0 0 0"/>
+    <origin xyz="0.3 0 0.9" rpy="0 0 0"/>
   </joint>
-  <!-- 显式传入参数 -->
-  <VLP-16 parent="base_link" name="velodyne" topic="/points_16" hz="10" samples="440" gpu="true">
-    <origin xyz="0.3 0 0.3" rpy="0 0 0" />
-  </VLP-16>
   <gazebo reference="velodyne_base_link">
-    <sensor type="ray" name="velodyne-VLP16">
+    <sensor type="gpu_ray" name="velodyne-VLP16">
       <pose>0 0 0 0 0 0</pose>
       <visualize>false</visualize>
@@ -186,7 +196,8 @@
         </range>
       </ray>
-      <plugin name="gazebo_ros_velodyne_laser_controller" filename="libgazebo_ros_velodyne_laser.so">
-        <topicName>/velodyne_points</topicName>
+      <plugin name="gazebo_ros_velodyne_laser" filename="libgazebo_ros_velodyne_laser.so">
+        <topicName>/points_16</topicName>
         <frameName>velodyne_base_link</frameName>
+        <organize_cloud>false</organize_cloud>
         <min_range>0.9</min_range>
         <max_range>130.0</max_range>
@@ -195,13 +206,8 @@
     </sensor>
   </gazebo>
-  <!-- ========================================================== -->
-  <!-- 6. Livox Mid-360 雷达 (车头中心点偏后0.1m) -->
-  <!-- ========================================================== -->
+  <!-- ============ 6. Livox Mid-360 雷达 ============ -->
   <xacro:include filename="$(find livox_laser_simulation)/urdf/livox_mid360.xacro"/>
-  <!-- 车头为 x=0.5, 往后偏0.1m，所以 x=0.4 -->
   <xacro:Livox_Mid40 name="livox" parent="base_link" xyz="0.4 0 0.45" rpy="3.1415926 0 0"/>
-  <!-- ========================================================== -->
-  <!-- 7. 差速驱动底盘插件 -->
-  <!-- ========================================================== -->
+  <!-- ============ 7. 差速驱动底盘插件 ============ -->
   <gazebo>
     <plugin name="differential_drive_controller" filename="libgazebo_ros_diff_drive.so">

Commit message: 修改16线雷达,避免16线雷达写法错误导致的gazebo崩溃

File: src/my_robot_description/urdf/robot.xacro (robot description, xacro)
@@ -158,5 +158,5 @@
   <xacro:corner_laser prefix="bright"  x="-0.5" y="-0.2" z="0.075" yaw="-2.356" />
   <!-- ============ 5. 16线激光雷达 (使用 GPU 版本 Velodyne 插件) ============ -->
-  <link name="velodyne_base_link">
+  <!-- <link name="velodyne_base_link">
     <xacro:cylinder_inertial mass="0.83" radius="0.0516" length="0.0717"/>
     <visual>
@@ -205,5 +205,5 @@
       </plugin>
     </sensor>
-  </gazebo>
+  </gazebo> -->
   <!-- ============ 6. Livox Mid-360 雷达 ============ -->
   <xacro:include filename="$(find livox_laser_simulation)/urdf/livox_mid360.xacro"/>

Commit message: 修改16线雷达

File: src/my_robot_description/urdf/robot.xacro (robot description, xacro)
@@ -72,4 +72,5 @@
       <parent link="base_link"/>
       <child link="${prefix}_wheel"/>
+      <!-- 轮子下沉 -0.05 使得底盘离地间隙合适 -->
       <origin xyz="-0.2 ${reflect * (base_width/2 + wheel_width/2)} -0.05" rpy="-1.5708 0 0"/>
       <axis xyz="0 0 1"/>
@@ -153,10 +154,11 @@
     </gazebo>
   </xacro:macro>
+  <!-- 部署四个单线雷达 -->
   <xacro:corner_laser prefix="left"    x="0.5"  y="0.2"  z="0.075" yaw="0.785" />
   <xacro:corner_laser prefix="right"   x="0.5"  y="-0.2" z="0.075" yaw="-0.785" />
   <xacro:corner_laser prefix="bleft"   x="-0.5" y="0.2"  z="0.075" yaw="2.356" />
   <xacro:corner_laser prefix="bright"  x="-0.5" y="-0.2" z="0.075" yaw="-2.356" />
-  <!-- ============ 5. 16线激光雷达 (使用 GPU 版本 Velodyne 插件) ============ -->
-  <!-- <link name="velodyne_base_link">
+  <!-- ============ 5. 16线激光雷达 (中心偏前0.3m处) ============ -->
+  <link name="velodyne">
     <xacro:cylinder_inertial mass="0.83" radius="0.0516" length="0.0717"/>
     <visual>
@@ -168,9 +170,10 @@
   <joint name="velodyne_base_mount_joint" type="fixed">
     <parent link="base_link"/>
-    <child link="velodyne_base_link"/>
-    <origin xyz="0.3 0 0.9" rpy="0 0 0"/>
+    <child link="velodyne"/>
+    <!-- 偏前0.3，置于底盘上方 z=0.8 处 -->
+    <origin xyz="0.3 0 0.8" rpy="0 0 0"/>
   </joint>
-  <gazebo reference="velodyne_base_link">
-    <sensor type="gpu_ray" name="velodyne-VLP16">
+  <gazebo reference="velodyne">
+    <sensor type="ray" name="velodyne-VLP16">
       <pose>0 0 0 0 0 0</pose>
       <visualize>false</visualize>
@@ -198,5 +201,5 @@
       <plugin name="gazebo_ros_velodyne_laser" filename="libgazebo_ros_velodyne_laser.so">
         <topicName>/points_16</topicName>
-        <frameName>velodyne_base_link</frameName>
+        <frameName>velodyne</frameName>
         <organize_cloud>false</organize_cloud>
         <min_range>0.9</min_range>
@@ -205,6 +208,7 @@
       </plugin>
     </sensor>
-  </gazebo> -->
-  <!-- ============ 6. Livox Mid-360 雷达 ============ -->
+  </gazebo>
+  <!-- ============ 6. Livox Mid-360 雷达 (车头中心点偏后0.1m) ============ -->
+  <!-- 车辆总长1.0，中心为0，车头为0.5。往后偏0.1就是 x=0.4 -->
   <xacro:include filename="$(find livox_laser_simulation)/urdf/livox_mid360.xacro"/>
   <xacro:Livox_Mid40 name="livox" parent="base_link" xyz="0.4 0 0.45" rpy="3.1415926 0 0"/>
@@ -224,5 +228,5 @@
       <odometryTopic>odom</odometryTopic>
       <odometryFrame>odom</odometryFrame>
-      <robotBaseFrame>base_link</robotBaseFrame>
+      <robotBaseFrame>base_footprint</robotBaseFrame> <!-- 修改这里为 base_footprint -->
       <publishWheelTF>false</publishWheelTF>
       <publishOdomTF>true</publishOdomTF>
